File: watch_hardware/page2.kicad_sch (KiCad schematic)
At the start: 36 parts, among them J2 TF_Card, Q1 PMOS, U7 LPS22HB, U8 CJC4344H, U9 OPA2192

Commit message: daily
Parts:
- MK1: footprint Connector_PinHeader_2.00mm:PinHeader_1x02_P2.00mm_Vertical -> Connector_PinHeader_1.00mm:PinHeader_1x02_P1.00mm_Vertical
Changed lines of the file:
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@@
 			)
 		)
-		(property "Footprint" "Connector_PinHeader_2.00mm:PinHeader_1x02_P2.00mm_Vertical"
+		(property "Footprint" "Connector_PinHeader_1.00mm:PinHeader_1x02_P1.00mm_Vertical"
 			(at 30.48 48.26 90)
 			(hide yes)
