File: watch_hardware/pwr.kicad_sch (KiCad schematic)
At the start: 43 parts, among them U13 TPS650250, U14 LM2664, U7 LM2664, U8 TP5000, U9 LM2664

Commit message: 原理图应该完成了吧……
Parts:
- removed U7, U9: LM2664, Package_TO_SOT_SMD:SOT-23-6, symbol projects:LM2664
- added C30, C36, C37: 10uF, Capacitor_SMD:C_0201_0603Metric, symbol Device:C
- added C31, C41: 100nF, Capacitor_SMD:C_0402_1005Metric, symbol Device:C
- C32: renamed from C16; footprint Capacitor_SMD:C_0402_1005Metric -> Capacitor_SMD:C_0201_0603Metric
- C33: renamed from C49; footprint Capacitor_SMD:C_0402_1005Metric -> Capacitor_SMD:C_0201_0603Metric
- C35: renamed from C50; footprint Capacitor_SMD:C_0402_1005Metric -> Capacitor_SMD:C_0201_0603Metric
- C38: renamed from C17; footprint Capacitor_SMD:C_0402_1005Metric -> Capacitor_SMD:C_0201_0603Metric
- C40: renamed from C46; footprint Capacitor_SMD:C_0402_1005Metric -> Capacitor_SMD:C_0201_0603Metric
- C42: renamed from C18; footprint Capacitor_SMD:C_0402_1005Metric -> Capacitor_SMD:C_0201_0603Metric
- C43: renamed from C48; footprint Capacitor_SMD:C_0402_1005Metric -> Capacitor_SMD:C_0201_0603Metric
- C45: renamed from C40; footprint Capacitor_SMD:C_0402_1005Metric -> Capacitor_SMD:C_0201_0603Metric
- C49: renamed from C42; footprint Capacitor_SMD:C_0402_1005Metric -> Capacitor_SMD:C_0201_0603Metric
- C51: renamed from C53; footprint Capacitor_SMD:C_0402_1005Metric -> Capacitor_SMD:C_0201_0603Metric
- C52: footprint Capacitor_SMD:C_0402_1005Metric -> Capacitor_SMD:C_0201_0603Metric
- C54: renamed from C45; footprint Capacitor_SMD:C_0402_1005Metric -> Capacitor_SMD:C_0201_0603Metric
- C56: renamed from C41; footprint Capacitor_SMD:C_0402_1005Metric -> Capacitor_SMD:C_0201_0603Metric
- renumbered C21 to C34, C51 to C39, C47 to C44, C28 to C46, C39 to C47, C43 to C48, C54 to C50, C44 to C53, C29 to C55, L3 to L1, L4 to L2, L2 to L3, L5 to L4, R23 to R25, R22 to R26, R24 to R27, R30 to R28, R28 to R30, R26 to R31, R27 to R32, R32 to R33, R31 to R34, U8 to U10, U14 to U11, U13 to U12
Connections:
- net +3.3V: now also U11.1 (V+), C30.1, C31.2
- net DCDC2: now also U11.4 (SD)
- net GND: now also U11.2 (GND), C30.2, C31.1, C36.1, C41.2
- net at U11.3 (CAP-): now also C37.2
- net -3V3: now reaches U11.5 (OUT)
- net -3V3: now also C36.2, C41.1
- net at U11.6 (CAP+): now also C37.1
Other:
- moved on the sheet: U11
