File: watch_hardware/pwr.kicad_sch (KiCad schematic)
At the start: 46 parts, among them U10 TP5000, U11 LM2664, U12 TPS650250

Commit message: 简单的画了了一下PCB
Parts:
- removed C39, C44, C50: 100nF, Capacitor_SMD:C_0402_1005Metric, symbol Device:C
- C30, C32, C33, C35, C36, C37, C38, C40, C42, C43, C45, C49, C51, C52, C54, C56: footprint Capacitor_SMD:C_0201_0603Metric -> Capacitor_SMD:C_0603_1608Metric
- R27: footprint Resistor_SMD:R_0603_1608Metric_Pad0.98x0.95mm_HandSolder -> Resistor_SMD:R_0402_1005Metric
Other:
- moved on the sheet: C33, C35, C40, C43
