File: watch_hardware/watch_hardware.kicad_sch (KiCad schematic)
At the start: 41 parts, among them J1 USB_C_Receptacle_USB2.0_16P, SW1 SW_Push, SW2 SW_Push, SW3 SW_Push, U1 ESP32-S3, U2 TK018F3716, U3 W25Q128JVP, U4 LIS3MDL, U5 LSM6DSOW, U6 AW9523B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

Commit message: 修改完电路
Connections:
- net GND: now also U2.25, U2.26, U2.27, U2.28
- no-connect marks 22 -> 18
Changed lines of the file:
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@@
+	)
+	(junction
+		(at 166.37 142.24)
+		(diameter 0)
+		(color 0 0 0 0)
 	)
 	(junction
@@
 	)
 	(junction
+		(at 171.45 157.48)
+		(diameter 0)
+		(color 0 0 0 0)
+	)
+	(junction
 		(at 219.71 143.51)
 		(diameter 0)
@@
 	)
 	(junction
+		(at 128.27 157.48)
+		(diameter 0)
+		(color 0 0 0 0)
+	)
+	(junction
 		(at 123.19 17.78)
 		(diameter 0)
@@
 	(junction
 		(at 33.02 72.39)
+		(diameter 0)
+		(color 0 0 0 0)
+	)
+	(junction
+		(at 135.89 142.24)
 		(diameter 0)
 		(color 0 0 0 0)
@@
 	)
 	(no_connect
-		(at 171.45 160.02)
-	)
-	(no_connect
 		(at 259.08 53.34)
 	)
@@
 	)
 	(no_connect
-		(at 128.27 157.48)
-	)
-	(no_connect
 		(at 152.4 97.79)
-	)
-	(no_connect
-		(at 171.45 157.48)
 	)
 	(no_connect
@@
 	)
 	(no_connect
-		(at 128.27 160.02)
-	)
-	(no_connect
 		(at 259.08 35.56)
 	)
@@
 	(wire
 		(pts
+			(xy 171.45 157.48) (xy 171.45 146.05)
+		)
+		(stroke
+			(width 0)
+			(type default)
+		)
+	)
+	(wire
+		(pts
 			(xy 104.14 49.53) (xy 71.12 49.53)
 		)
@@
 	(wire
 		(pts
-			(xy 163.83 142.24) (xy 168.91 142.24)
+			(xy 163.83 142.24) (xy 166.37 142.24)
 		)
 		(stroke
@@
 	(wire
 		(pts
+			(xy 171.45 160.02) (xy 171.45 157.48)
+		)
+		(stroke
+			(width 0)
+			(type default)
+		)
+	)
+	(wire
+		(pts
 			(xy 247.65 135.89) (xy 259.08 135.89)
 		)
@@
 	(wire
 		(pts
+			(xy 171.45 146.05) (xy 166.37 146.05)
+		)
+		(stroke
+			(width 0)
+			(type default)
+		)
+	)
+	(wire
+		(pts
 			(xy 158.75 139.7) (xy 138.43 139.7)
 		)
@@
 	(wire
 		(pts
+			(xy 128.27 160.02) (xy 128.27 157.48)
+		)
+		(stroke
+			(width 0)
+			(type default)
+		)
+	)
+	(wire
+		(pts
 			(xy 259.08 58.42) (xy 274.32 58.42)
 		)
@@
 	(wire
 		(pts
+			(xy 128.27 157.48) (xy 128.27 142.24)
+		)
+		(stroke
+			(width 0)
+			(type default)
+		)
+	)
+	(wire
+		(pts
 			(xy 19.05 25.4) (xy 19.05 72.39)
 		)
@@
 	(wire
 		(pts
+			(xy 166.37 142.24) (xy 168.91 142.24)
+		)
+		(stroke
+			(width 0)
+			(type default)
+		)
+	)
+	(wire
+		(pts
 			(xy 129.54 97.79) (xy 129.54 107.95)
 		)
@@
 	(wire
 		(pts
+			(xy 166.37 146.05) (xy 166.37 142.24)
+		)
+		(stroke
+			(width 0)
+			(type default)
+		)
+	)
+	(wire
+		(pts
 			(xy 29.21 87.63) (xy 33.02 87.63)
 		)
@@
 		)
 		(stroke
+			(width 0)
+			(type default)
+		)
+	)
+	(wire
+		(pts
+			(xy 128.27 142.24) (xy 135.89 142.24)
+		)
+		(stroke
