File: watch_hardware/watch_hardware.kicad_pcb (KiCad board)
At the start: 4 copper layers, 31.7 x 39.6 mm, 130 parts, among them J1 USB_C_Receptacle_USB2.0_16P, J2 TF_Card, SW1 SW_Push, SW2 SW_Push, SW3 SW_Push, SW4 SW_Push, U1 ESP32-S3, U10 TP5000, U11 LM2664, U12 TPS650250, U2 TK018F3716, U3 W25Q128JVP, U4 LIS3MDL, U5 LSM6DSOW, U6 AW9523B, U7 LPS22HB, U8 CJC4344H, U9 OPA2192, Y1 Crystal_GND24

Commit message: daily
Parts:
- removed the C1 at (152.1, 80.0)
- removed the C35 at (143.2, 50.2)
- removed C45, C49, C50, C51, C53, C55: 10uF, Capacitor_SMD:C_0603_1608Metric
- removed C46, C48, C52, C54: 100nF, Capacitor_SMD:C_0402_1005Metric
- removed C47: 1uF, Capacitor_SMD:C_0402_1005Metric
- removed the C9 at (113.8, 67.2)
- removed the D2 at (149.6, 78.3)
- removed L5: 2.2uH, Inductor_SMD:L_Changjiang_FTC201610S
- removed the R1 at (151.1, 79.9)
- removed R10: 680k, Resistor_SMD:R_0402_1005Metric_Pad0.72x0.64mm_HandSolder
- removed the R13 at (99.2, 66.8)
- removed the R14 at (99.2, 68.8)
- removed the R16 at (99.2, 72.8)
- removed the R17 at (99.2, 74.8)
- removed R27: 10k, Resistor_SMD:R_0402_1005Metric_Pad0.72x0.64mm_HandSolder
- removed R28: 500m, Resistor_SMD:R_0402_1005Metric
- removed R29, R31, R33, R34, R9: 100k, Resistor_SMD:R_0402_1005Metric_Pad0.72x0.64mm_HandSolder
- removed R30, R35: 22k, Resistor_SMD:R_0402_1005Metric_Pad0.72x0.64mm_HandSolder
- removed R32: 1R0, Resistor_SMD:R_0402_1005Metric_Pad0.72x0.64mm_HandSolder
- removed the R7 at (148.1, 77.6)
- removed the R8 at (95.9, 74.8)
- removed the SW1 at (151.7, 82.1)
- removed the U10 at (146.4, 51.0)
- removed U12: TPS650250, Package_DFN_QFN:QFN-32-1EP_5x5mm_P0.5mm_EP3.6x3.6mm_ThermalVias
- added C37: 10uF, Capacitor_SMD:C_0603_1608Metric, F.Cu at (98.6, 56.3)
- added C38: 10uF, Capacitor_SMD:C_0603_1608Metric, F.Cu at (98.6, 51.3)
- added C41: 10uF, Capacitor_SMD:C_0603_1608Metric, F.Cu at (98.6, 43.7)
- added Q1: PMOS, Package_TO_SOT_SMD:SOT-23, B.Cu at (161.4, 66.0)
- added R21: 10k, Resistor_SMD:R_0402_1005Metric_Pad0.72x0.64mm_HandSolder, F.Cu at (105.9, 39.9)
- added R22: 10k, Resistor_SMD:R_0402_1005Metric_Pad0.72x0.64mm_HandSolder, F.Cu at (105.9, 37.9)
- added R6: 10k, Resistor_SMD:R_0402_1005Metric_Pad0.72x0.64mm_HandSolder, F.Cu at (145.2, 63.1)
- added SW4: SW_Push, Connector_PinHeader_1.00mm:PinHeader_1x02_P1.00mm_Vertical, F.Cu at (105.9, 42.5)
- added U11: TPS65217, Package_DFN_QFN:VQFN-48-1EP_6x6mm_P0.4mm_EP4.1x4.1mm_ThermalVias, F.Cu at (128.0, 48.9)
- C34: value 10uF -> 100nF; footprint Capacitor_SMD:C_0603_1608Metric -> Capacitor_SMD:C_0402_1005Metric
- C8: value 10uF -> 1uF; footprint Capacitor_SMD:C_0603_1608Metric -> Capacitor_SMD:C_0402_1005Metric
- J1: moved to B.Cu
- L2: value 4.7uH -> 2.2uH
- R18: renamed from R24; value 100 -> 50
- R20: renamed from R26; value 5.6k -> 75k
- moved C40 60.7 mm to (98.6, 36.2), turned to 0 degrees
- moved C43 59.6 mm to (98.6, 46.2), turned to 0 degrees
- moved L3 58.3 mm to (102.4, 40.0)
- moved L4 58.3 mm to (102.4, 43.3)
- moved C36 57.8 mm to (98.6, 53.8), turned to 0 degrees
- moved C44 57.8 mm to (98.6, 48.8), turned to 0 degrees
- moved C42 56.4 mm to (98.6, 41.2), turned to 0 degrees
- moved C39 55.1 mm to (98.6, 38.7), turned to 0 degrees
- moved L2 51.6 mm to (102.4, 36.6)
- moved C4 42.5 mm to (155.6, 56.4)
- moved LS1 42.3 mm to (150.9, 81.7)
- moved C6 41.6 mm to (155.1, 57.7)
- moved C8 30.9 mm to (144.7, 64.6), turned to 90 degrees
- moved C30 21.8 mm to (129.1, 57.6)
- moved C32 21.8 mm to (136.5, 60.0)
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- renumbered C2 to C1, C12 to C10, C13 to C11, C14 to C12, C15 to C13, C16 to C14, C17 to C15, C18 to C16, C19 to C17, C20 to C18, C21 to C19, C3 to C2, C22 to C20, C23 to C21, C24 to C22, C25 to C23, C26 to C24, C27 to C25, C28 to C26, C29 to C27, C30 to C28, C31 to C29, C4 to C3, C32 to C30, C33 to C31, C37 to C32, C38 to C33, C41 to C35, C5 to C4, C6 to C5, C7 to C6, C10 to C7, C11 to C9, D11 to D10, D3 to D2, D4 to D3, D5 to D4, D6 to D5, D7 to D6, D8 to D7, D9 to D8, D10 to D9, R2 to R1, R15 to R11, R18 to R12, R19 to R13, R20 to R14, R21 to R15, R22 to R16, R23 to R17, R25 to R19, R3 to R2, R4 to R3, R5 to R4, R6 to R5, R11 to R7, R12 to R8, SW2 to SW1, SW3 to SW2, SW4 to SW3, U11 to U10
Connections:
- BT1 pad 1: /BAT -> Net-(BT1-+)
- C1 pad 1: /GPIO0 -> /GPIO1
- C25 pad 1: +3.3V -> +3.3VDAC
- C26 pad 1: +3.3V -> +3.3VDAC
- C34 pad 1: +5V -> GND
- C34 pad 2: GND -> +5V
- C36 pad 2: +3.3VA -> +5V
- C39 pad 1: Net-(U10-VS) -> GND
- C39 pad 2: GND -> Net-(U11-VDCDC1)
- C40 pad 2: +3.3VA -> Net-(U11-VDCDC1)
- C42 pad 1: Net-(U10-VS) -> +3V3
- C43 pad 1: +3V3 -> GND
- C43 pad 2: GND -> +1V0
- C44 pad 1: +3V3 -> GND
- C44 pad 2: GND -> +1V0
- L2 pad 1: Net-(L2-Pad1) -> Net-(U11-VDCDC1)
- L2 pad 2: Net-(U10-VS) -> Net-(U11-L1)
- L3 pad 1: +3.3VA -> +3V3
- L4 pad 1: +3V3 -> Net-(U11-L3)
- L4 pad 2: Net-(U12-L1) -> +1V0
- R1 pad 1: /GPIO0 -> /GPIO1
- R20 pad 1: Net-(U10-TS) -> Net-(U11-TS)
- R20 pad 2: +5V -> GND
- SW1 pad 1: /GPIO0 -> /GPIO1
- TH1 pad 1: GND -> Net-(U11-TS)
- TH1 pad 2: Net-(U10-TS) -> GND
- U1 pad 11: Net-(U1-GPIO6) -> /MUX_OUT
- U1 pad 13: /SDA1 -> /PWR_EN
- U1 pad 14: /SCL1 -> unconnected-(U1-GPIO9-Pad14)
- U1 pad 22: /L_TE -> /L_INT
- U1 pad 23: /L_INT -> /AW_INT
- U1 pad 24: /AW_INT -> unconnected-(U1-GPIO18-Pad24)
- U1 pad 37: /TF_DAT1 -> /TF_CMD
- U1 pad 38: /TF_DAT0 -> /TF_DAT3
- U1 pad 39: /TF_CLK -> /TF_DAT2
- U1 pad 40: /TF_CMD -> /TF_DAT1
- U1 pad 41: /TF_DAT3 -> /TF_DAT0
- U1 pad 42: /TF_DAT2 -> /TF_CLK
- U1 pad 5: /GPIO0 -> /PMIC_INT
- U10 pad 4: /DCDC2 -> +3.3V
- U2 pad 14: /L_TE -> unconnected-(U2-Pad14)
- U4 pad 1: /SCL1 -> /SCL0
- U4 pad 11: /SDA1 -> /SDA0
- U5 pad 13: /SCL1 -> /SCL0
- U5 pad 14: /SDA1 -> /SDA0
- U6 pad 11: /LIS_DRDY -> unconnected-(U6-P0_5-Pad11)
- U6 pad 14: /DCDC3 -> unconnected-(U6-P1_4-Pad14)
- U6 pad 17: unconnected-(U6-P1_7-Pad17) -> /TF_CD
- U6 pad 2: /MIC_P -> unconnected-(U6-P1_1-Pad2)
- U6 pad 3: /TF_CD -> unconnected-(U6-P1_2-Pad3)
- U6 pad 4: /DCDC2 -> /LIS_DRDY
- U6 pad 5: /CHRG -> /L_RST
- U6 pad 6: /STDBY -> unconnected-(U6-P0_1-Pad6)
- U6 pad 7: /L_RST -> /T_RST
- U6 pad 8: /T_RST -> unconnected-(U6-P0_3-Pad8)
- U8 pad 9: +3.3V -> +3.3VDAC
Routing:
- net /TF_CD: track 0.00 -> 31.0 mm
- net /USB_D+: track 0.00 -> 23.4 mm, vias 0 -> 1
- net /USB_D-: track 0.00 -> 23.2 mm, vias 0 -> 2
- net +3V3: track 0.00 -> 21.5 mm, vias 2 -> 7
- net /TF_DAT1: track 0.00 -> 21.0 mm
- net /L_MOSI: track 0.00 -> 18.9 mm, vias 0 -> 2
- net /TF_DAT2: track 0.00 -> 18.0 mm
- net /TF_DAT0: track 0.00 -> 15.4 mm
- net /TF_DAT3: track 0.00 -> 15.2 mm
- net /TF_CLK: track 0.00 -> 14.8 mm
- net /TF_CMD: track 0.00 -> 14.6 mm
- net /L_D1: track 0.00 -> 13.8 mm, vias 0 -> 2
- net /L_SCK: track 0.00 -> 13.7 mm, vias 0 -> 2
- net /L_D3: track 0.00 -> 13.2 mm, vias 0 -> 2
- net /L_D2: track 0.00 -> 12.0 mm, vias 0 -> 2
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