File: watch_hardware/watch_hardware.kicad_pcb (KiCad board)
At the start: 4 copper layers, 31.7 x 39.6 mm, 119 parts, among them J1 USB_C_Receptacle_USB2.0_16P, J2 TF_Card, Q1 PMOS, SW1 SW_Push, SW2 SW_Push, SW3 SW_Push, SW4 SW_Push, U1 ESP32-S3, U10 MAX2769C, U11 LM2664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

Commit message: 修改完电路
Parts:
- moved C35 0.11 mm to (159.5, 76.2)
- moved C41 0.10 mm to (166.6, 71.6)
- moved D9 0.05 mm to (158.6, 69.7)
Connections:
- U2 pad 25: unconnected-(U2-Pad25) -> GND
- U2 pad 26: unconnected-(U2-Pad26) -> GND
- U2 pad 27: unconnected-(U2-Pad27) -> GND
- U2 pad 28: unconnected-(U2-Pad28) -> GND
Routing:
- net /SCL0: track 111.6 -> 118.3 mm
- net +3.3VADC: track 103.4 -> 108.3 mm, vias 7 -> 8
- net GND: track 44.3 -> 39.9 mm, vias 148 -> 152
- net +3V3: track 228.4 -> 232.4 mm, vias 18 -> 19
- net /AW_INT: track 12.7 -> 15.3 mm
- net Net-(U10-LNAOUT): track 6.31 -> 8.31 mm
- net /LIS_DRDY: track 32.0 -> 33.9 mm
- net /PWR_EN: track 23.3 -> 25.1 mm
- net /MAX_I1: track 33.5 -> 31.9 mm
- net Net-(U10-MIXIN): track 2.93 -> 1.51 mm
- net /GPIO1: track 33.0 -> 31.9 mm
- net +3.3V: track 55.9 -> 54.8 mm
- net /L_SCK: track 25.8 -> 26.9 mm
- net /L_MOSI: track 22.6 -> 23.5 mm
- net +3.3VP: track 74.9 -> 74.1 mm
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
Commit message: 修改了电路，以符合生产需求
Parts:
- J1: footprint Connector_USB:USB_C_Receptacle_HRO_TYPE-C-31-M-12 -> projects:usb_C_16p
- moved J1 0.40 mm to (170.4, 65.1)
Routing:
- net /SCL0: track 118.3 -> 121.2 mm
